File: hardware/BoardModules/PSU/PSU.kicad_pcb (KiCad board)
At the start: 2 copper layers, 44.5 x 25.4 mm, 27 parts, among them P1 INPUT, P2 CONN_01X03, P3 PWR_SW, P4 OUTPUT, Q1 P, U1 MCP73831, U2 LT1308

Commit message: More hardware
Parts:
- added REF**: PinHeader_1x01_P2.54mm_Vertical, Connector_PinHeader_2.54mm:PinHeader_1x01_P2.54mm_Vertical, F.Cu at (158.8, 102.9)
- added REF**: PinHeader_1x01_P2.54mm_Vertical, Connector_PinHeader_2.54mm:PinHeader_1x01_P2.54mm_Vertical, F.Cu at (156.2, 102.9)
- added REF**: PinHeader_1x01_P2.54mm_Vertical, Connector_PinHeader_2.54mm:PinHeader_1x01_P2.54mm_Vertical, F.Cu at (156.2, 80.0)
- added REF**: PinHeader_1x01_P2.54mm_Vertical, Connector_PinHeader_2.54mm:PinHeader_1x01_P2.54mm_Vertical, F.Cu at (158.8, 80.0)
- LED1: value Red -> R
- LED2: value Green -> G
- R9: value 49k -> 47k
- U1: value MCP73831 -> 73831
Other:
- board size 44.5 x 25.4 mm -> 45.7 x 25.4 mm
- board text added: "1.3"
- board text added: "PSU module r1.3 Angry Wasp © 2022"
- board text removed: "1.2"
