File: hardware/BoardModules/Propeller/Propeller.kicad_pcb (KiCad board)
At the start: 2 copper layers, 35.6 x 53.3 mm, 36 parts, among them P1 CONN_01X02, P10 CONN_01X02, P11 CONN_01X02, P12 CONN_01X02, P13 CONN_01X02, P14 CONN_01X02, P15 CONN_01X02, P16 CONN_01X02, P17 CONN_01X02, P18 CONN_01X02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

Commit message: More hardware
Parts:
- removed REF**: PinHeader_1x20_P2.54mm_Vertical, Connector_PinHeader_2.54mm:PinHeader_1x20_P2.54mm_Vertical
Connections:
- P28 pad 1: 2A -> 1A
- P28 pad 2: 1A -> 2A
- U1 pad 31: 2Y -> 1Y
- U1 pad 32: 1Y -> 2Y
Routing:
- net 1A: track 13.7 -> 17.1 mm
- net 2A: track 13.1 -> 14.1 mm
- net 2Y: track 15.1 -> 15.9 mm
- net SDA: track 45.3 -> 44.8 mm
Other:
- board text added: "3v3"
- board text added: "5v input"
- board text added: "A1"
- board text added: "A2"
- board text added: "A3"
- board text added: "A4"
- board text added: "A5"
- board text added: "A6"
- board text added: "A7"
- board text added: "A8"
- board text added: "ADC"
- board text added: "GND"
- board text added: "I2C"
- board text added: "NC"
- board text added: "P10"
- board text added: "P11"
- board text added: "P12"
- board text added: "P13"
- board text added: "P14"
- board text added: "P15"
- board text added: "P16"
- board text added: "P17"
- board text added: "P18"
- board text added: "P19"
- board text added: "P20"
- board text added: "P21"
- board text added: "P22"
- board text added: "P23"
- board text added: "P24"
- board text added: "P25"
- board text added: "P26"
- board text added: "P27"
- board text added: "P4"
- board text added: "P5"
- board text added: "P6"
- board text added: "P7"
- board text added: "P8"
- board text added: "P9"
- board text added: "Prop Module r1.4 Angry Wasp © 2022"
- board text added: "RESn"
- board text added: "RX"
- board text added: "SCL"
- board text added: "SDA"
- board text added: "TX"
- board text added: "UART"
- board text removed: "angrywasp.net.au rev 1.4"
